File: B115R_bass_preamp/B115R_bass_preamp.sch (KiCad schematic (older format))
At the start: 66 parts, among them J1 Line in, J2 Line out, SW1 On/Bypass, SW2 Ultra Hi, SW3 Ultra Lo

Commit message: v2
Parts:
- removed C18: 100nF, symbol Device:C
- added C18: 22µF 50V, Capacitor_THT:CP_Axial_L11.0mm_D6.0mm_P18.00mm_Horizontal, symbol Device:CP
- added Trimpot: A1M, Potentiometer_THT:Potentiometer_Piher_PC-16_Single_Horizontal, symbol Device:R_POT
- C14: footprint Capacitor_THT:C_Axial_L22.0mm_D10.5mm_P27.50mm_Horizontal -> Capacitor_THT:C_Axial_L19.0mm_D7.5mm_P25.00mm_Horizontal
- C6: value 33nF -> 33nF 50V
- R1, R14, R19, R2: value 1.5K 0.5W -> 1.5K 1W
- R25: value 1M -> 100K 1W; Links (none) -> https://www.tube-town.net/ttstore/xicon-carbon-film-resisto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; Power (none) -> 1W
- R26: value 1.5K -> 1M; Links (none) -> https://www.tube-town.net/ttstore/xicon-carbon-film-resisto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
- R27: value 100K -> 1.5K 1W
- R33: Links (none) -> https://www.tube-town.net/ttstore/xicon-carbon-film-resisto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
- renumbered Bass1 to Bass, Gain1 to Gain, HiMid1 to HiMid, LowMid1 to LowMid, Treble1 to Treble, Volume1 to Volume
Connections:
- net GND: now also R26.2, C18.2, Trimpot.1
- net VCC: now also R25.1; no longer V2.6 (A)
- net at Volume.2: now also R26.1, V2.7 (G)
- net at C8.1: now also Trimpot.3; no longer R23.2
- net at V2.8 (K): now also R27.1, C18.1; no longer R26.1
- net at C14.2, R25.2: now also V2.6 (A); no longer R26.2, R27.1
- new net: R23.2, Trimpot.2
Other:
- note added: "Active Tonestack"
- note added: "Driver\nStage"
- note added: "Filter"
- note added: "Ultra High\nBypass capacitor"
- note added: "Ultra Low\nTonestack"
- note added: "Voltage\nDropping"
- moved on the sheet: C10, C12, C6, C8, C9, R14, R15, R2, Volume
